File: hardware/light-strip/light-strip.kicad_pcb (KiCad board)
At the start: 2 copper layers, 270 x 10 mm, 11 parts, among them J1 Conn_01x01, J2 Conn_01x01

Commit message: Add a second set of pad for symetrical connect Update PCB and ajust size with housing Add 2 mounting holes, just in case Add fabrication files.
Parts:
- added J1: -, Connector_Wire:SolderWirePad_1x01_SMD_5x10mm, F.Cu at (278.6, 113.0)
- added J2: +, Connector_Wire:SolderWirePad_1x01_SMD_5x10mm, F.Cu at (278.6, 108.0)
- added REF**: MountingHole_3.2mm_M3, MountingHole:MountingHole_3.2mm_M3, F.Cu at (194.5, 110.0)
- added REF**: MountingHole_3.2mm_M3, MountingHole:MountingHole_3.2mm_M3, F.Cu at (104.5, 110.0)
- J3: renamed from J1; value Conn_01x01 -> -
- J4: renamed from J2; value Conn_01x01 -> +
Routing:
- net Net-(D1-Pad1): track 197.3 -> 274.9 mm
- net Net-(D3-Pad2): track 259.7 -> 275.0 mm
Other:
- board size 270 x 10 mm -> 270 x 12.4 mm
